Commit message: Rename my_robot for diff_robot

File: diff_robot_description/urdf/camera.xacro (robot description, xacro)
@@ -1,4 +1,4 @@
 <?xml version='1.0'?>
-<robot name="my_robot" xmlns:xacro="http://www.ros.org/wiki/xacro">
+<robot name="diff_robot" xmlns:xacro="http://www.ros.org/wiki/xacro">
 <xacro:macro name="my_cam" params="x:=0 y:=0 z:=0">
     <link name="camera">

File: diff_robot_description/urdf/caster_wheel.xacro (robot description, xacro)
@@ -1,4 +1,4 @@
 <?xml version='1.0'?>
-<robot name="my_robot" xmlns:xacro="http://www.ros.org/wiki/xacro">
+<robot name="diff_robot" xmlns:xacro="http://www.ros.org/wiki/xacro">
 <xacro:macro name="caster_wheel" params="radius mass x:=0 y:=0 z:=0">
     <link name='caster_wheel'>

File: diff_robot_description/urdf/chassis.xacro (robot description, xacro)
@@ -1,4 +1,4 @@
 <?xml version='1.0'?>
-<robot name="my_robot" xmlns:xacro="http://www.ros.org/wiki/xacro">
+<robot name="diff_robot" xmlns:xacro="http://www.ros.org/wiki/xacro">
 <xacro:macro name="box_chassis" params="length width height mass">
   <link name='chassis'>

File: diff_robot_description/urdf/diff_robot.xacro (robot description, xacro)
@@ -1,4 +1,4 @@
 <?xml version='1.0'?>
-<robot name="my_robot" xmlns:xacro="http://www.ros.org/wiki/xacro">
+<robot name="diff_robot" xmlns:xacro="http://www.ros.org/wiki/xacro">
   <!-- Chassis properties-->
   <xacro:property name="chassis_length" value="0.4"/>
@@ -17,17 +17,17 @@
   <xacro:property name="wheel_z" value="0"/>
   <!-- Import the chassis of the robot -->
-  <xacro:include filename="$(find my_robot_description)/urdf/chassis.xacro" />
+  <xacro:include filename="$(find diff_robot_description)/urdf/chassis.xacro" />
   <!-- Import a macro which constructs a spheric caster wheel -->
-  <xacro:include filename="$(find my_robot_description)/urdf/caster_wheel.xacro" />
+  <xacro:include filename="$(find diff_robot_description)/urdf/caster_wheel.xacro" />
   <!-- Import a macro which constructs a wheel -->
-  <xacro:include filename="$(find my_robot_description)/urdf/wheel.xacro" />
+  <xacro:include filename="$(find diff_robot_description)/urdf/wheel.xacro" />
   <!-- Import the camera attached to the chassis -->
-  <xacro:include filename="$(find my_robot_description)/urdf/camera.xacro" />
+  <xacro:include filename="$(find diff_robot_description)/urdf/camera.xacro" />
   <!-- Import the hokuyo Lidar  -->
-  <xacro:include filename="$(find my_robot_description)/urdf/hokuyo.xacro" />
+  <xacro:include filename="$(find diff_robot_description)/urdf/hokuyo.xacro" />
     <!-- Import colors for Rviz -->
-  <xacro:include filename="$(find my_robot_description)/urdf/materials.xacro" />
+  <xacro:include filename="$(find diff_robot_description)/urdf/materials.xacro" />
   <!-- Import all Gazebo-customization elements (plugins and colors) -->
-  <xacro:include filename="$(find my_robot_description)/urdf/my_robot.gazebo"/>
+  <xacro:include filename="$(find diff_robot_description)/urdf/diff_robot.gazebo"/>
   <!-- The base_footprint is the representation of the robot position with respect to the origin
       of the world. The base_footprint link is a virtual (non-physical) link which has no dimensions

File: diff_robot_description/urdf/hokuyo.xacro (robot description, xacro)
@@ -1,4 +1,4 @@
 <?xml version='1.0'?>
-<robot name="my_robot" xmlns:xacro="http://www.ros.org/wiki/xacro">
+<robot name="diff_robot" xmlns:xacro="http://www.ros.org/wiki/xacro">
 <xacro:macro name="hokuyo" params="x:=0 y:=0 z:=0">
     <link name="hokuyo">
@@ -11,5 +11,5 @@
             <origin xyz="0.0 0.0 0.0" rpy="0.0 0.0 0.0"/>
             <geometry>
-                <mesh filename="package://my_robot_description/meshes/hokuyo.dae"/>
+                <mesh filename="package://diff_robot_description/meshes/hokuyo.dae"/>
             </geometry>
             <material name="">

File: diff_robot_description/urdf/materials.xacro (robot description, xacro)
@@ -1,4 +1,4 @@
 <?xml version='1.0'?>
-<robot name="my_robot" xmlns:xacro="http://www.ros.org/wiki/xacro">
+<robot name="diff_robot" xmlns:xacro="http://www.ros.org/wiki/xacro">
   <material name="black">
     <color rgba="0.0 0.0 0.0 1.0"/>

File: diff_robot_description/urdf/wheel.xacro (robot description, xacro)
@@ -1,4 +1,4 @@
 <?xml version='1.0'?>
-<robot name="my_robot" xmlns:xacro="http://www.ros.org/wiki/xacro">
+<robot name="diff_robot" xmlns:xacro="http://www.ros.org/wiki/xacro">
 <xacro:macro name="wheel" params="side mass x:=0 y:=0 z:=0 radius length">
     <xacro:property name="reflect" value="1"/>

Commit message: Fix inertias and collisions

File: diff_robot_description/urdf/camera.xacro (robot description, xacro)
@@ -1,34 +1,31 @@
 <?xml version='1.0'?>
 <robot name="diff_robot" xmlns:xacro="http://www.ros.org/wiki/xacro">
-<xacro:macro name="my_cam" params="x:=0 y:=0 z:=0">
+<xacro:macro name="cam" params="mass size x:=0 y:=0 z:=0">
     <link name="camera">
-        <inertial>
-            <origin xyz="0.0 0.0 0.0" rpy="0.0 0.0 0.0"/>
-            <mass value="0.1"/>
-            <inertia ixx="1e-6" ixy="0.0" ixz="0.0" iyy="1e-6" iyz="0.0" izz="1e-6"/>
-        </inertial>
         <visual name="">
-            <origin xyz="0.0 0.0 0.0" rpy="0.0 0.0 0.0"/>
+            <origin xyz="0 0 0" rpy="0 0 0"/>
             <geometry>
-                <box size="0.05 0.05 0.05"/>
+                <box size="${size} ${size} ${size}"/>
             </geometry>
-            <material name="">
-                <color rgba="0 0.0 0.0 1.0"/>
-                <texture filename=""/>
-            </material>
+            <!-- Color For Rviz-->
+            <material name="black"/>
         </visual>
         <collision>
-            <origin xyz="0.0 0.0 0.0" rpy="0.0 0.0 0.0"/>
+            <origin xyz="0 0 0" rpy="0 0 0"/>
             <geometry>
-                <box size="0.05 0.05 0.05"/>
+                <box size="${size} ${size} ${size}"/>
             </geometry>
         </collision>
+        <inertial>
+            <origin xyz="0 0 0" rpy="0 0 0"/>
+            <mass value="${mass}"/>
+            <xacro:box_inertia m="${mass}" x="${size}" y="${size}" z="${size}"/>
+        </inertial>
     </link>
     <joint name="camera_joint" type="fixed">
-        <origin xyz="${x} ${y} ${z}" rpy="0.0 0.0 0.0"/>
+        <origin xyz="${x} ${y} ${z}" rpy="0 0 0"/>
         <parent link="chassis"/>
         <child link="camera"/>
-        <axis xyz="0.0 1 0.0"/>
-        <limit lower="0.0" upper="0.0" effort="0.0" velocity="0.0"/>
+        <axis xyz="0 1 0"/>
     </joint>
 </xacro:macro>

File: diff_robot_description/urdf/caster_wheel.xacro (robot description, xacro)
@@ -3,25 +3,23 @@
 <xacro:macro name="caster_wheel" params="radius mass x:=0 y:=0 z:=0">
     <link name='caster_wheel'>
+        <visual>
+            <origin xyz="0 0 0" rpy=" 0 0 0"/>
+            <geometry>
+                <sphere radius="${radius}"/>
+            </geometry>
+            <!-- Color For Rviz-->
+            <material name="black"/>
+        </visual>
+        <collision>
+            <origin xyz="0 0 0" rpy=" 0 0 0"/>
+            <geometry>
+                <sphere radius="${radius}"/>
+            </geometry>
+        </collision>
         <inertial>
             <mass value="${mass}"/>
             <origin xyz="0.0 0 0" rpy=" 0 0 0"/>
-            <inertia
-                ixx="${mass*radius*radius*2/5}" ixy="0" ixz="0"
-                iyy="${mass*radius*radius*2/5}" iyz="0"
-                izz="${mass*radius*radius*2/5}"
-            />
+            <xacro:sphere_inertia m="${mass}" r="${radius}"/>
         </inertial>
-        <collision>
-            <origin xyz="0 0 0" rpy=" 0 0 0"/>
-            <geometry>
-            <sphere radius="${radius}"/>
-            </geometry>
-        </collision>
-        <visual>
-            <origin xyz="0 0 0" rpy=" 0 0 0"/>
-            <geometry>
-            <sphere radius="${radius}"/>
-            </geometry>
-        </visual>
     </link>
     <joint name="caster_wheel_joint" type="fixed">

File: diff_robot_description/urdf/chassis.xacro (robot description, xacro)
@@ -3,13 +3,12 @@
 <xacro:macro name="box_chassis" params="length width height mass">
   <link name='chassis'>
-    <inertial>
-      <mass value="${mass}"/>
-      <origin xyz="0.0 0 0" rpy=" 0 0 0"/>
-      <inertia
-          ixx="${(mass/12)*(width*width+height*height)}" ixy="0" ixz="0"
-          iyy="${(mass/12)*(length*length+height*height)}" iyz="0"
-          izz="${(mass/12)*(width*width+length*length)}"
-      />
-    </inertial>
+    <visual>
+      <origin xyz="0 0 0" rpy=" 0 0 0"/>
+      <geometry>
+        <box size="${length} ${width} ${height}"/>
+      </geometry>
+      <!-- Color For Rviz-->
+      <material name="green"/>
+    </visual>
     <collision>
       <origin xyz="0 0 0" rpy=" 0 0 0"/>
@@ -18,13 +17,11 @@
       </geometry>
     </collision>
-    <visual>
-      <origin xyz="0 0 0" rpy=" 0 0 0"/>
-      <geometry>
-        <box size="${length} ${width} ${height}"/>
-      </geometry>
-    </visual>
+    <inertial>
+      <mass value="${mass}"/>
+      <origin xyz="0.0 0 0" rpy=" 0 0 0"/>
+      <xacro:box_inertia m="${mass}" x="${width}" y="${length}" z="${height}"/>
+    </inertial>
   </link>
   <joint name="robot_footprint_joint" type="fixed">
-    <origin xyz="0 0 ${height/2} " rpy="0 0 0" />
     <parent link="robot_footprint"/>
     <child link="chassis" />

File: diff_robot_description/urdf/diff_robot.xacro (robot description, xacro)
@@ -16,4 +16,7 @@
   <xacro:property name="wheel_y" value="${chassis_width/2 + wheel_length/2 + 0.01}"/>
   <xacro:property name="wheel_z" value="0"/>
+  <!-- camera properties -->
+  <xacro:property name="cam_mass" value="0.1"/>
+  <xacro:property name="cam_size" value="0.05"/>
   <!-- Import the chassis of the robot -->
   <xacro:include filename="$(find diff_robot_description)/urdf/chassis.xacro" />
@@ -26,6 +29,8 @@
   <!-- Import the hokuyo Lidar  -->
   <xacro:include filename="$(find diff_robot_description)/urdf/hokuyo.xacro" />
-    <!-- Import colors for Rviz -->
+  <!-- Import colors for Rviz -->
   <xacro:include filename="$(find diff_robot_description)/urdf/materials.xacro" />
+  <!-- Import inertia macros -->
+  <xacro:include filename="$(find diff_robot_description)/urdf/inertias.xacro" />
   <!-- Import all Gazebo-customization elements (plugins and colors) -->
   <xacro:include filename="$(find diff_robot_description)/urdf/diff_robot.gazebo"/>
@@ -45,5 +50,5 @@
   <xacro:wheel side="right"  mass="${wheel_mass}" x="${wheel_x}" y="${wheel_y}" z="${wheel_z}" radius="${wheel_radius}" length="${wheel_length}"/>
   <!-- Camera -->
-  <xacro:my_cam x="${chassis_length/2}"/>
+  <xacro:cam mass="${cam_mass}" size="${cam_size}" x="${chassis_length/2}"/>
   <!-- Lidar -->
   <xacro:hokuyo x="${chassis_length/4}" z="${chassis_height/2 + 0.05}"/>

File: diff_robot_description/urdf/hokuyo.xacro (robot description, xacro)
@@ -3,32 +3,27 @@
 <xacro:macro name="hokuyo" params="x:=0 y:=0 z:=0">
     <link name="hokuyo">
-        <inertial>
-            <origin xyz="0.0 0.0 0.0" rpy="0.0 0.0 0.0"/>
-            <mass value="1e-5"/>
-            <inertia ixx="1e-6" ixy="0.0" ixz="0.0" iyy="1e-6" iyz="0.0" izz="1e-6"/>
-        </inertial>
         <visual name="">
-            <origin xyz="0.0 0.0 0.0" rpy="0.0 0.0 0.0"/>
+            <origin xyz="0 0 0" rpy="0 0 0"/>
             <geometry>
                 <mesh filename="package://diff_robot_description/meshes/hokuyo.dae"/>
             </geometry>
-            <material name="">
-                <color rgba="0 0.0 0.0 1.0"/>
-                <texture filename=""/>
-            </material>
         </visual>
         <collision>
-            <origin xyz="0.0 0.0 0.0" rpy="0.0 0.0 0.0"/>
+            <origin xyz="0 0 0" rpy="0 0 0"/>
             <geometry>
-                <box size="0.1 0.1 0.1"/>
+                <mesh filename="package://diff_robot_description/meshes/hokuyo.dae"/>
             </geometry>
         </collision>
+        <inertial>
+            <origin xyz="0 0 0" rpy="0 0 0"/>
+            <mass value="0.1"/>
+            <xacro:box_inertia m="0.1" x="0.05" y="0.05" z="0.05"/>
+        </inertial>
     </link>
     <joint name="hokuyo_joint" type="fixed">
-        <origin xyz="${x} ${y} ${z}" rpy="0.0 0.0 0.0"/>
+        <origin xyz="${x} ${y} ${z}" rpy="0 0 0"/>
         <parent link="chassis"/>
         <child link="hokuyo"/>
-        <axis xyz="0.0 1 0.0"/>
-        <limit lower="0.0" upper="0.0" effort="0.0" velocity="0.0"/>
+        <axis xyz="0 1 0"/>
     </joint>
 </xacro:macro>

File: diff_robot_description/urdf/materials.xacro (robot description, xacro)
@@ -8,5 +8,5 @@
   </material>
   <material name="green">
-    <color rgba="0.0 0.8 0.0 1.0"/>
+    <color rgba="0.48 0.93 0.69 1.0"/>
   </material>
   <material name="grey">

File: diff_robot_description/urdf/wheel.xacro (robot description, xacro)
@@ -7,25 +7,23 @@
     </xacro:if>
     <link name="${side}_wheel">
-        <inertial>
-            <origin xyz="0.0 0.0 0.0" rpy="0.0 1.5707 1.5707"/>
-            <mass value="${mass}"/>
-            <inertia
-                ixx="${(mass/12)*(3*radius*radius+length*length)}" ixy="0.0" ixz="0.0"
-                iyy="${(mass/12)*(3*radius*radius+length*length)}" iyz="0.0"
-                izz="${(mass/2)*(radius*radius)}"
-            />
-        </inertial>
         <visual name="${side}_wheel_visual">
-            <origin xyz="0.0 0 0" rpy="0.0 1.5707 1.5707"/>
+            <origin xyz="0 0 0" rpy="${pi/2} 0 0"/>
             <geometry>
                 <cylinder radius="${radius}" length="${length}"/>
             </geometry>
+            <!-- Color For Rviz-->
+            <material name="black"/>
         </visual>
         <collision name="${side}_wheel_collision">
-            <origin xyz="0.0 0 0" rpy="0.0 1.5707 1.5707"/>
+            <origin xyz="0 0 0" rpy="${pi/2} 0 0"/>
             <geometry>
                 <cylinder radius="${radius}" length="${length}"/>
             </geometry>
         </collision>
+        <inertial>
+            <origin xyz="0 0 0" rpy="${pi/2} 0 0"/>
+            <mass value="${mass}"/>
+            <xacro:cylinder_inertia m="${mass}" r="${radius}" h="${length}"/>
+        </inertial>
     </link>
     <joint name="${side}_wheel_hinge" type="continuous">
