Commit message: Add properties and friction for caster wheel

File: diff_robot_description/urdf/diff_robot.xacro (robot description, xacro)
@@ -2,18 +2,20 @@
 <robot name="diff_robot" xmlns:xacro="http://www.ros.org/wiki/xacro">
   <!-- Chassis properties-->
-  <xacro:property name="chassis_length" value="0.3"/>
+  <xacro:property name="chassis_length" value="0.4"/>
   <xacro:property name="chassis_width" value="0.2"/>
   <xacro:property name="chassis_height" value="0.1"/>
-  <xacro:property name="chassis_mass" value="15"/>
-  <!-- Caster Wheel properties-->
-  <xacro:property name="caster_mass" value="0.2"/>
-  <xacro:property name="caster_radius" value="0.05"/>
+  <xacro:property name="chassis_mass" value="5"/>
   <!-- Wheel properties-->
   <xacro:property name="wheel_radius" value="0.1"/>
   <xacro:property name="wheel_length" value="0.05"/>
   <xacro:property name="wheel_mass" value="5"/>
-  <xacro:property name="wheel_x" value="${chassis_length/4}"/>
+  <xacro:property name="wheel_x" value="0.07"/>
   <xacro:property name="wheel_y" value="${chassis_width/2 + wheel_length/2}"/>
   <xacro:property name="wheel_z" value="0"/>
+  <!-- Caster Wheel properties-->
+  <xacro:property name="caster_mass" value="3"/>
+  <xacro:property name="caster_radius" value="${wheel_radius/2}"/>
+  <xacro:property name="caster_x" value="${-chassis_length/4}"/>
+  <xacro:property name="caster_z" value="${-caster_radius}"/>
   <!-- camera properties -->
   <xacro:property name="cam_mass" value="0.1"/>
@@ -33,6 +35,6 @@
   <!-- Import inertia macros -->
   <xacro:include filename="$(find diff_robot_description)/urdf/inertias.xacro" />
-  <!-- The base_footprint is the representation of the robot position with respect to the origin
-      of the world. The base_footprint link is a virtual (non-physical) link which has no dimensions
+  <!-- The base_link is the representation of the robot position with respect to the origin
+      of the world. The base_link link is a virtual (non-physical) link which has no dimensions
       or collision areas. Its primary purpose is to enable various packages determine the center
       of a robot projected to the ground. For example, Navigation2 uses this link to determine the
@@ -42,5 +44,5 @@
   <xacro:box_chassis length="${chassis_length}" width="${chassis_width}" height="${chassis_height}" mass="${chassis_mass}"/>
   <!-- Caster wheel -->
-  <xacro:caster_wheel radius="${caster_radius}" mass="${caster_mass}" x="-0.1" z="-0.05"/>
+  <xacro:caster_wheel radius="${caster_radius}" mass="${caster_mass}" x="${caster_x}" z="${caster_z}"/>
   <!-- Back Left wheel -->
   <xacro:wheel side="left"   mass="${wheel_mass}" x="${wheel_x}" y="${wheel_y}" z="${wheel_z}" radius="${wheel_radius}" length="${wheel_length}"/>
@@ -50,5 +52,5 @@
   <xacro:cam mass="${cam_mass}" size="${cam_size}" x="${chassis_length/2}"/>
   <!-- Lidar -->
-  <xacro:hokuyo x="${chassis_length/4}" z="${chassis_height/2 + 0.05}"/>
+  <xacro:hokuyo x="${chassis_length/4}" z="${chassis_height/2 + 0.04}"/>
   <!-- INCLUDE THIS AT THE END -->
   <!-- Import all Gazebo-customization elements (plugins and colors) -->
