Commit message: Add robot control for gazebo

File: diff_robot_description/urdf/chassis.xacro (robot description, xacro)
@@ -24,5 +24,5 @@
   </link>
   <joint name="robot_footprint_joint" type="fixed">
-    <parent link="robot_footprint"/>
+    <parent link="base_link"/>
     <child link="chassis" />
   </joint>

File: diff_robot_description/urdf/diff_robot.xacro (robot description, xacro)
@@ -2,5 +2,5 @@
 <robot name="diff_robot" xmlns:xacro="http://www.ros.org/wiki/xacro">
   <!-- Chassis properties-->
-  <xacro:property name="chassis_length" value="0.4"/>
+  <xacro:property name="chassis_length" value="0.3"/>
   <xacro:property name="chassis_width" value="0.2"/>
   <xacro:property name="chassis_height" value="0.1"/>
@@ -14,5 +14,5 @@
   <xacro:property name="wheel_mass" value="5"/>
   <xacro:property name="wheel_x" value="${chassis_length/4}"/>
-  <xacro:property name="wheel_y" value="${chassis_width/2 + wheel_length/2 + 0.01}"/>
+  <xacro:property name="wheel_y" value="${chassis_width/2 + wheel_length/2}"/>
   <xacro:property name="wheel_z" value="0"/>
   <!-- camera properties -->
@@ -33,6 +33,4 @@
   <!-- Import inertia macros -->
   <xacro:include filename="$(find diff_robot_description)/urdf/inertias.xacro" />
-  <!-- Import all Gazebo-customization elements (plugins and colors) -->
-  <xacro:include filename="$(find diff_robot_description)/urdf/diff_robot.gazebo"/>
   <!-- The base_footprint is the representation of the robot position with respect to the origin
       of the world. The base_footprint link is a virtual (non-physical) link which has no dimensions
@@ -40,5 +38,5 @@
       of a robot projected to the ground. For example, Navigation2 uses this link to determine the
       center of a circular footprint used in its obstacle avoidance algorithms-->
-  <link name="robot_footprint"/>
+  <link name="base_link"/>
   <!-- Chassis -->
   <xacro:box_chassis length="${chassis_length}" width="${chassis_width}" height="${chassis_height}" mass="${chassis_mass}"/>
@@ -53,3 +51,6 @@
   <!-- Lidar -->
   <xacro:hokuyo x="${chassis_length/4}" z="${chassis_height/2 + 0.05}"/>
+  <!-- INCLUDE THIS AT THE END -->
+  <!-- Import all Gazebo-customization elements (plugins and colors) -->
+  <xacro:include filename="$(find diff_robot_description)/urdf/diff_robot.gazebo"/>
 </robot>

File: diff_robot_description/urdf/wheel.xacro (robot description, xacro)
@@ -27,5 +27,5 @@
         </inertial>
     </link>
-    <joint name="${side}_wheel_hinge" type="continuous">
+    <joint name="${side}_wheel_joint" type="continuous">
         <origin xyz="${x} ${reflect*y} ${z}" rpy="0.0 0.0 0.0"/>
         <parent link="chassis"/>
@@ -33,7 +33,4 @@
         <axis xyz="0.0 1 0.0"/>
     </joint>
-    <gazebo reference="${side}_wheel">
-        <material>Gazebo/Black </material>
-    </gazebo>
 </xacro:macro>
 </robot>

Commit message: Fix chassis inertia

File: diff_robot_description/urdf/chassis.xacro (robot description, xacro)
@@ -19,9 +19,10 @@
     <inertial>
       <mass value="${mass}"/>
-      <origin xyz="0.0 0 0" rpy=" 0 0 0"/>
-      <xacro:box_inertia m="${mass}" x="${width}" y="${length}" z="${height}"/>
+      <origin xyz="${length/4} 0 0" rpy=" 0 0 0"/>
+      <xacro:box_inertia m="${mass}" x="${length}" y="${width}" z="${height}" xd="${length/4}"/>
     </inertial>
   </link>
-  <joint name="robot_footprint_joint" type="fixed">
+  <joint name="chassis_joint" type="fixed">
+    <origin xyz="${-length/4} 0 0" rpy="0 0 0"/>
     <parent link="base_link"/>
     <child link="chassis" />

File: diff_robot_description/urdf/inertias.xacro (robot description, xacro)
@@ -7,8 +7,8 @@
     />
   </xacro:macro>
-  <xacro:macro name="box_inertia" params="m x y z">
-    <inertia  ixx="${m*(y*y+z*z)/12}" ixy = "0" ixz = "0"
-      iyy="${m*(x*x+z*z)/12}" iyz = "0"
-      izz="${m*(x*x+z*z)/12}"
+  <xacro:macro name="box_inertia" params="m x y z xd:=0 yd:=0 zd:=0">
+    <inertia  ixx="${m*(y*y+z*z)/12 + m*xd*xd}" ixy = "0" ixz = "0"
+      iyy="${m*(x*x+z*z)/12 + m*yd*yd}" iyz = "0"
+      izz="${m*(x*x+z*z)/12 + m*zd*zd}"
     />
   </xacro:macro>

Commit message: Stabilize robot in simulation

File: diff_robot_description/urdf/chassis.xacro (robot description, xacro)
@@ -1,5 +1,5 @@
 <?xml version='1.0'?>
 <robot name="diff_robot" xmlns:xacro="http://www.ros.org/wiki/xacro">
-<xacro:macro name="box_chassis" params="length width height mass">
+<xacro:macro name="box_chassis" params="length width height mass z_rot_axis:=${[0,0]}">
   <link name='chassis'>
     <visual>
@@ -19,10 +19,10 @@
     <inertial>
       <mass value="${mass}"/>
-      <origin xyz="${length/4} 0 0" rpy=" 0 0 0"/>
-      <xacro:box_inertia m="${mass}" x="${length}" y="${width}" z="${height}" xd="${length/4}"/>
+      <origin xyz="${z_rot_axis[0]} 0 0" rpy=" 0 0 0"/>
+      <xacro:box_inertia m="${mass}" x="${length}" y="${width}" z="${height}" xd="${z_rot_axis[0]}" yd="${z_rot_axis[1]}"/>
     </inertial>
   </link>
   <joint name="chassis_joint" type="fixed">
-    <origin xyz="${-length/4} 0 0" rpy="0 0 0"/>
+    <origin xyz="${-z_rot_axis[0]} 0 0" rpy="0 0 0"/>
     <parent link="base_link"/>
     <child link="chassis" />

File: diff_robot_description/urdf/diff_robot.xacro (robot description, xacro)
@@ -42,5 +42,5 @@
   <link name="base_link"/>
   <!-- Chassis -->
-  <xacro:box_chassis length="${chassis_length}" width="${chassis_width}" height="${chassis_height}" mass="${chassis_mass}"/>
+  <xacro:box_chassis length="${chassis_length}" width="${chassis_width}" height="${chassis_height}" mass="${chassis_mass}" z_rot_axis="${[wheel_x, 0]}"/>
   <!-- Caster wheel -->
   <xacro:caster_wheel radius="${caster_radius}" mass="${caster_mass}" x="${caster_x}" z="${caster_z}"/>
@@ -52,5 +52,5 @@
   <xacro:cam mass="${cam_mass}" size="${cam_size}" x="${chassis_length/2}"/>
   <!-- Lidar -->
-  <xacro:hokuyo x="${chassis_length/4}" z="${chassis_height/2 + 0.04}"/>
+  <xacro:hokuyo x="${wheel_x}" z="${chassis_height/2 + 0.05}"/>
   <!-- INCLUDE THIS AT THE END -->
   <!-- Import all Gazebo-customization elements (plugins and colors) -->

File: diff_robot_description/urdf/wheel.xacro (robot description, xacro)
@@ -2,7 +2,8 @@
 <robot name="diff_robot" xmlns:xacro="http://www.ros.org/wiki/xacro">
 <xacro:macro name="wheel" params="side mass x:=0 y:=0 z:=0 radius length">
-    <xacro:property name="reflect" value="1"/>
+    <!-- Right wheel is on the negative y axis -->
+    <xacro:property name="reflect" value="-1"/>
     <xacro:if value="${side.endswith('left')}">
-        <xacro:property name="reflect" value="-1"/>
+        <xacro:property name="reflect" value="1"/>
     </xacro:if>
     <link name="${side}_wheel">
